Commit message: feat: simulate in gazebo;

File: urdf/robot.urdf (robot description, URDF)
Before this commit: robot my_robot, 6 links, 5 joints
Links:
- link base_link: geometry collision box size=0.8 0.6 0.25; visual box size=1 0.6 0.25
- link front_left_wheel_link: geometry collision cylinder length=0.1 radius=0.15; visual cylinder length=0.1 radius=0.15
- link front_right_wheel_link: geometry collision cylinder length=0.1 radius=0.15; visual cylinder length=0.1 radius=0.15
- link rear_left_wheel_link: geometry collision cylinder length=0.1 radius=0.15; visual cylinder length=0.1 radius=0.15
- link rear_right_wheel_link: geometry collision cylinder length=0.1 radius=0.15; visual cylinder length=0.1 radius=0.15
Joints:
- joint base_to_camera: origin xyz=0 0 0.325 rpy=0 0 0 -> xyz=0 0 0.45 rpy=0 0 0
- joint base_to_front_left_wheel: origin xyz=0.25 0.34 0.1 rpy=1.57075 0 0 -> xyz=0.3 0.35 0.15 rpy=1.57075 0 0
- joint base_to_front_right_wheel: origin xyz=0.25 -0.34 0.1 rpy=1.57075 0 0 -> xyz=0.3 -0.35 0.15 rpy=1.57075 0 0
- joint base_to_rear_left_wheel: origin xyz=-0.25 0.34 0.1 rpy=1.57075 0 0 -> xyz=-0.3 0.35 0.15 rpy=1.57075 0 0
- joint base_to_rear_right_wheel: origin xyz=-0.25 -0.34 0.1 rpy=1.57075 0 0 -> xyz=-0.3 -0.35 0.15 rpy=1.57075 0 0

Commit message: feat: opencv;

File: urdf/robot.urdf (robot description, URDF)
Before this commit: robot my_robot, 6 links, 5 joints
Links:
- link base_link: mass 5.0 -> None; geometry collision box size=1 0.6 0.25; visual box size=1 0.6 0.25
- link camera_link: mass 0.2 -> 3.0
- link front_left_wheel_link: mass 0.5 -> 2.0
- link front_right_wheel_link: mass 0.5 -> 2.0
- link rear_left_wheel_link: mass 0.5 -> 2.0
- link rear_right_wheel_link: mass 0.5 -> 2.0

Commit message: feat: camera;

File: urdf/robot.urdf (robot description, URDF)
Before this commit: robot my_robot, 6 links, 5 joints
Joints:
- joint base_to_camera: origin xyz=0 0 0.45 rpy=0 0 0 -> xyz=0.4 0 0.45 rpy=0 0 0
